Commit message: Laser scanner - implementation

File: urdf/barista_robot_model.urdf (robot description, URDF)
Before this commit: robot barista_robot, 15 links, 14 joints
Links:
- removed link center_base_link
- removed link center_column_link
- added link laser_link, mass 0.2; collision cylinder length=0.04 radius=0.055; visual mesh filename=package://barista_robot_description/meshes/slamtec_rplidar_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
Joints:
- removed joint center_base_joint
- removed joint center_column_joint
- added joint laser_joint: type fixed, parent chassis, child laser_link, origin xyz=0 0 0.185 rpy=0 0 0
